Commit message: Switched from skid steer to ackerman

File: my_robot/urdf/MSE6_robot.xacro (robot description, xacro)
@@ -11,10 +11,10 @@
         <pose>0 0 0 0 0 0</pose>
         <inertial>
-            <mass value="5.0"/>
+            <mass value="3.0"/>
             <origin xyz="0 0 .01" rpy="0 0 0"/>
             <inertia
-                ixx="0.0112" ixy="0" ixz="0"
-                iyy="0.0445" iyz="0"
-                izz="0.0417"
+                ixx="0.0067" ixy="0" ixz="0"
+                iyy="0.0267" iyz="0"
+                izz="0.025"
                 />
         </inertial>
@@ -32,5 +32,28 @@
         </visual>
     </link>
-    <link name="right_wheel">
+    <link name="front_right_strut">
+        <collision>
+            <origin xyz="0 0 0" rpy="0 0 0"/>
+            <geometry>
+                <box size="0.01 0.005 0.015"/>
+            </geometry>
+        </collision>
+        <inertial>
+            <origin xyz="0 0 0" rpy="0 0 0"/>
+            <mass value="1e-5"/>
+            <inertia
+                ixx="1e-6" ixy="0" ixz="0"
+                iyy="1e-6" iyz="0"
+                izz="1e-6"
+                />
+        </inertial>
+        <visual>
+            <origin xyz="0 0 0" rpy="0 0 0"/>
+            <geometry>
+               <box size="0.01 0.005 0.015"/>
+            </geometry>
+        </visual>
+    </link>
+    <link name="front_right_wheel">
         <collision>
             <origin xyz="0 0 0" rpy="0 1.5707 1.5707"/>
@@ -38,12 +61,4 @@
                 <cylinder radius="0.025" length="0.015"/>
             </geometry>
-            <surface>
-                <friction>
-                    <ode>
-                        <mu>1</mu>
-                        <mu2>0.01</mu2>
-                    </ode>
-                </friction>
-            </surface>
         </collision>
         <inertial>
@@ -51,7 +66,7 @@
             <origin xyz="0 0 0" rpy="0 1.5707 1.5707"/>
             <inertia
-            ixx="0.1" ixy="0" ixz="0"
-            iyy="0.1" iyz="0"
-            izz="0.1"
+            ixx="0.000018" ixy="0" ixz="0"
+            iyy="0.000018" iyz="0"
+            izz="0.000031"
             />
         </inertial>
@@ -63,5 +78,28 @@
         </visual>
     </link>
-    <link name="rr_wheel">
+    <link name="rear_right_strut">
+        <collision>
+            <origin xyz="0 0 0" rpy="0 0 0"/>
+            <geometry>
+                <box size="0.01 0.01 0.025"/>
+            </geometry>
+        </collision>
+        <inertial>
+            <origin xyz="0 0 0" rpy="0 0 0"/>
+            <mass value="1e-5"/>
+            <inertia
+                ixx="1e-6" ixy="0" ixz="0"
+                iyy="1e-6" iyz="0"
+                izz="1e-6"
+                />
+        </inertial>
+        <visual>
+            <origin xyz="0 0 0" rpy="0 0 0"/>
+            <geometry>
+               <box size="0.01 0.01 0.025"/>
+            </geometry>
+        </visual>
+    </link>
+    <link name="rear_right_wheel">
         <collision>
             <origin xyz="0 0 0" rpy="0 1.5707 1.5707"/>
@@ -69,12 +107,4 @@
                 <cylinder radius="0.030" length="0.015"/>
             </geometry>
-            <surface>
-                <friction>
-                    <ode>
-                        <mu>1</mu>
-                        <mu2>0.01</mu2>
-                    </ode>
-                </friction>
-            </surface>
         </collision>
         <inertial>
@@ -82,7 +112,7 @@
             <origin xyz="0 0 0" rpy="0 1.5707 1.5707"/>
             <inertia
-            ixx="0.1" ixy="0" ixz="0"
-            iyy="0.1" iyz="0"
-            izz="0.1"
+               ixx="0.000024" ixy="0" ixz="0"
+               iyy="0.000024" iyz="0"
+               izz="0.000045"
             />
         </inertial>
@@ -94,5 +124,28 @@
         </visual>
     </link>
-    <link name="left_wheel">
+    <link name="front_left_strut">
+        <collision>
+            <origin xyz="0 0 0" rpy="0 0 0"/>
+            <geometry>
+                <box size="0.01 0.005 0.015"/>
+            </geometry>
+        </collision>
+        <inertial>
+            <origin xyz="0 0 0" rpy="0 0 0"/>
+            <mass value="1e-5"/>
+            <inertia
+                ixx="1e-6" ixy="0" ixz="0"
+                iyy="1e-6" iyz="0"
+                izz="1e-6"
+                />
+        </inertial>
+        <visual>
+            <origin xyz="0 0 0" rpy="0 0 0"/>
+            <geometry>
+               <box size="0.01 0.005 0.015"/>
+            </geometry>
+        </visual>
+    </link>
+    <link name="front_left_wheel">
         <collision>
             <origin xyz="0 0 0" rpy="0 1.5707 1.5707"/>
@@ -100,12 +153,4 @@
                 <cylinder radius="0.025" length="0.015"/>
             </geometry>
-            <surface>
-                <friction>
-                    <ode>
-                        <mu>1</mu>
-                        <mu2>0.01</mu2>
-                    </ode>
-                </friction>
-            </surface>
         </collision>
         <inertial>
@@ -113,7 +158,7 @@
             <origin xyz="0 0 0" rpy="0 1.5707 1.5707"/>
             <inertia
-            ixx="0.1" ixy="0" ixz="0"
-            iyy="0.1" iyz="0"
-            izz="0.1"
+               ixx="0.000018" ixy="0" ixz="0"
+               iyy="0.000018" iyz="0"
+               izz="0.000031"
             />
         </inertial>
@@ -124,6 +169,29 @@
             </geometry>
         </visual>
-    </link>
-    <link name="lr_wheel">
+     </link>
+    <link name="rear_left_strut">
+        <collision>
+            <origin xyz="0 0 0" rpy="0 0 0"/>
+            <geometry>
+                <box size="0.01 0.01 0.025"/>
+            </geometry>
+        </collision>
+        <inertial>
+            <origin xyz="0 0 0" rpy="0 0 0"/>
+            <mass value="1e-5"/>
+            <inertia
+                ixx="1e-6" ixy="0" ixz="0"
+                iyy="1e-6" iyz="0"
+                izz="1e-6"
+                />
+        </inertial>
+        <visual>
+            <origin xyz="0 0 0" rpy="0 0 0"/>
+            <geometry>
+               <box size="0.01 0.01 0.025"/>
+            </geometry>
+        </visual>
+    </link>
+    <link name="rear_left_wheel">
         <collision>
             <origin xyz="0 0 0" rpy="0 1.5707 1.5707"/>
@@ -131,12 +199,4 @@
                 <cylinder radius="0.030" length="0.015"/>
             </geometry>
-            <surface>
-                <friction>
-                    <ode>
-                        <mu>1</mu>
-                        <mu2>0.01</mu2>
-                    </ode>
-                </friction>
-            </surface>
         </collision>
         <inertial>
@@ -144,7 +204,7 @@
             <origin xyz="0 0 0" rpy="0 1.5707 1.5707"/>
             <inertia
-            ixx="0.1" ixy="0" ixz="0"
-            iyy="0.1" iyz="0"
-            izz="0.1"
+               ixx="0.000024" ixy="0" ixz="0"
+               iyy="0.000024" iyz="0"
+               izz="0.000045"
             />
         </inertial>
@@ -156,14 +216,14 @@
         </visual>
     </link>
-        <gazebo reference="left_wheel">
+        <gazebo reference="front_left_wheel">
             <material>Gazebo/Black</material>
         </gazebo>
-        <gazebo reference="right_wheel">
+        <gazebo reference="front_right_wheel">
             <material>Gazebo/Black</material>
         </gazebo>
-        <gazebo reference="lr_wheel">
+        <gazebo reference="rear_left_wheel">
             <material>Gazebo/Black</material>
         </gazebo>
-        <gazebo reference="rr_wheel">
+        <gazebo reference="rear_right_wheel">
             <material>Gazebo/Black</material>
         </gazebo>
@@ -174,32 +234,60 @@
             <material>Gazebo/Blue</material>
         </gazebo>
-    <joint name="left_wheel_hinge" type="continuous">
-        <origin xyz="0.09 0.067 -.05" rpy="0 0 0"/>
-        <child link="left_wheel"/>
-        <parent link="chassis"/>
+    <joint name="front_left_steer_bearing" type="revolute">
+        <origin xyz="0.09 0.057 -.079" rpy="0 0 0"/>
+        <child link="front_left_strut"/>
+        <parent link="chassis"/>
+        <axis xyz="0 0 1" rpy="0 0 0"/>
+        <limit effort="50" velocity="1.0" lower="-0.3" upper="0.3"/>
+    </joint>
+    <joint name="front_left_wheel_bearing" type="continuous">
+        <origin xyz="0 .011 0.01" rpy="0 0 0"/>
+        <child link="front_left_wheel"/>
+        <parent link="front_left_strut"/>
         <axis xyz="0 1 0" rpy="0 0 0"/>
         <limit effort="100" velocity="100"/>
+    </joint>
+    <joint name="front_right_steer_bearing" type="revolute">
+        <origin xyz="0.09 -0.057 -.079" rpy="0 0 0"/>
+        <child link="front_right_strut"/>
+        <parent link="chassis"/>
+        <axis xyz="0 0 1" rpy="0 0 0"/>
+        <limit effort="50" velocity="1.0" lower="-0.3" upper="0.3"/>
+    </joint>
+    <joint name="front_right_wheel_bearing" type="continuous">
+        <origin xyz="0 -.011 0.01" rpy="0 0 0"/>
+        <child link="front_right_wheel"/>
+        <parent link="front_right_strut"/>
+        <axis xyz="0 1 0" rpy="0 0 0"/>
+        <limit effort="100" velocity="100"/>
+    </joint>
+    <joint name="rear_left_steer_bearing" type="fixed">
+        <origin xyz="-0.09 0.067 -.053" rpy="0 0 0"/>
+        <child link="rear_left_strut"/>
+        <parent link="chassis"/>
+        <axis xyz="0 0 1" rpy="0 0 0"/>
+        <limit effort="100" velocity="100"/>
         <dynamics damping=".0" friction=".00"/>
     </joint>
-    <joint name="right_wheel_hinge" type="continuous">
-        <origin xyz="0.09 -0.067 -.05" rpy="0 0 0"/>
-        <child link="right_wheel"/>
-        <parent link="chassis"/>
+    <joint name="rear_left_wheel_bearing" type="continuous">
+        <origin xyz="0 0 0" rpy="0 0 0"/>
+        <child link="rear_left_wheel"/>
+        <parent link="rear_left_strut"/>
         <axis xyz="0 1 0" rpy="0 0 0"/>
         <limit effort="100" velocity="100"/>
         <dynamics damping=".0" friction=".00"/>
     </joint>
-    <joint name="lr_wheel_hinge" type="continuous">
-        <origin xyz="-0.09 0.067 -.06" rpy="0 0 0"/>
-        <child link="lr_wheel"/>
-        <parent link="chassis"/>
-        <axis xyz="0 1 0" rpy="0 0 0"/>
+    <joint name="rear_right_steer_bearing" type="fixed">
+        <origin xyz="-0.09 -0.067 -.053" rpy="0 0 0"/>
+        <child link="rear_right_strut"/>
+        <parent link="chassis"/>
+        <axis xyz="0 0 1" rpy="0 0 0"/>
         <limit effort="100" velocity="100"/>
         <dynamics damping=".0" friction=".00"/>
     </joint>
-    <joint name="rr_wheel_hinge" type="continuous">
-        <origin xyz="-0.09 -0.067 -.06" rpy="0 0 0"/>
-        <child link="rr_wheel"/>
-        <parent link="chassis"/>
+    <joint name="rear_right_wheel_bearing" type="continuous">
+        <origin xyz="0 0 0" rpy="0 0 0"/>
+        <child link="rear_right_wheel"/>
+        <parent link="rear_right_strut"/>
         <axis xyz="0 1 0" rpy="0 0 0"/>
         <limit effort="100" velocity="100"/>
